File: Daughterboard/SDCard.kicad_sch (KiCad schematic)
At the start: 8 parts, among them J7 Micro_SD_Card_Det, U11 TXB0104D

Commit message: fixed part no.s for availability
Parts:
- C44, C45: Distrib Part No. 1276-1000-1-ND -> (none); Distrib. Name Digi-Key -> (none)
