File: Daughterboard/RUST_Daughterboard.kicad_sch (KiCad schematic)
At the start: 37 parts, among them J1 Conn_Coaxial, J2 SIM, J3 Conn_01x12, J6 Conn_01x12, K1 EE2-3TNU-L

Commit message: fixed part no.s for availability
Parts:
- J2: 2nd Chc. Mfg. Name AVX Corp. -> (none); 2nd Chc. Part No. 009162006301150 -> (none)
- MH1, MH2, MH4: now left out of the parts list
- MH3: value M2 SMT NUT -> MountingHole; footprint MyFootprints:SMTSO-M2-3ET -> MountingHole:MountingHole_2.2mm_M2; Mfg. Name PEM -> (none); Mfg. Part No. SMTSO-M2-3ET -> (none); now left out of the parts list
Other:
- note added: "3/3/25 P/N CHANGES FOR ASSEMBLY HOUSE -J2 (SIM connector): WILL SEND -L1 (high Q 2.4nH): New P/N listed. -L2 (high Q 12nH): New P/N listed. -L4 (high Q 9.1nH): New P/N listed. -Can select alt parts for inductors as long as they're high-Q. Remove M2 nut"
- note removed: "NOTE: POPULATING AUDIO TVS from Mainboard for Ds here"
- moved on the sheet: MH1, MH2, MH3, MH4

Commit message: for phase 1 prod
Parts:
- AE1: Notes (none) -> Can send.
- J2: Notes (none) -> Will send.
Other:
- note added: "3/3/25 P/N CHANGES FOR ASSEMBLY HOUSE -J2 (SIM connector): WILL SEND -L1 (high Q 2.4nH): New P/N listed. -L2 (high Q 12nH): New P/N listed. -L4 (high Q 9.1nH): New P/N listed. -Can select alt parts for inductors as long as they're high-Q. Removed M2 nut"
- note removed: "3/3/25 P/N CHANGES FOR ASSEMBLY HOUSE -J2 (SIM connector): WILL SEND -L1 (high Q 2.4nH): New P/N listed. -L2 (high Q 12nH): New P/N listed. -L4 (high Q 9.1nH): New P/N listed. -Can select alt parts for inductors as long as they're high-Q. Remove M2 nut"
Changed lines of the file:
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@@
 		)
 	)
-	(text "3/3/25 P/N CHANGES FOR ASSEMBLY HOUSE\n\n-J2 (SIM connector): WILL SEND\n-L1 (high Q 2.4nH): New P/N listed.\n-L2 (high Q 12nH): New P/N listed.\n-L4 (high Q 9.1nH): New P/N listed.\n-Can select alt parts for inductors as long as they're high-Q. \n\nRemove M2 nut"
+	(text "3/3/25 P/N CHANGES FOR ASSEMBLY HOUSE\n\n-J2 (SIM connector): WILL SEND\n-L1 (high Q 2.4nH): New P/N listed.\n-L2 (high Q 12nH): New P/N listed.\n-L4 (high Q 9.1nH): New P/N listed.\n-Can select alt parts for inductors as long as they're high-Q. \n\nRemoved M2 nut"
 		(exclude_from_sim no)
 		(at 267.462 44.704 0)
@@
 			)
 		)
+		(property "Notes" "Will send."
+			(at 274.955 204.47 0)
+			(effects
+				(font
+					(size 1.27 1.27)
+				)
+				(hide yes)
+			)
+		)
 		(pin "1"
 		)
@@
 			(at 257.175 103.505 0)
 			(effects
+				(font
+					(size 1.27 1.27)
+				)
+				(hide yes)
+			)
+		)
+		(property "Notes" "Can send."
+			(at 257.175 103.505 0)
+			(effects
