File: Dialboard/RUST_Dialboard.kicad_pcb (KiCad board)
At the start: 2 copper layers, 53 x 39 mm, 10 parts, among them U1 HallSwitch

Commit message: for phase 1 prod
Other:
- board text added: "Fab notes: -Thickness: 2.4mm -Solder mask: Black -Surface finish: ENIG or whatever"
- board text removed: "Fab notes: -Thickness: 2.4mm -Solder mask: Color not important, but preference for black? -Surface finish: ENIG or whatever"
Changed lines of the file:
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@@
 		)
 	)
-	(gr_text "Fab notes:\n	-Thickness: 2.4mm\n	-Solder mask: Color not important, but preference for black?\n	-Surface finish: ENIG or whatever"
+	(gr_text "Fab notes:\n	-Thickness: 2.4mm\n	-Solder mask: Black\n	-Surface finish: ENIG or whatever"
 		(at 99.912 60 0)
 		(layer "Cmts.User")
