File: Motherboard/CellTranceiver.kicad_sch (KiCad schematic)
At the start: 32 parts, among them J11 U.FL, J13 U.FL, J14 U.FL, J15 U.FL, J16 U.FL, J4 U.FL, J5 U.FL, Q1 NMOS DMG2302UK-7, Q2 NMOS DMG2302UK-7, T1 TestPoint_Alt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

Commit message: changed file names
Parts:
- Q1, Q2: value NMOS DMG2302UK-7 -> NMOS DMG2302UK-7
