File: Motherboard/RUST_Motherboard.kicad_sch (KiCad schematic)
At the start: 52 parts, among them J3 12p Male Samtec Connector, J6 12p Male Samtec Connector, J7 Conn_02x03_Counter_Clockwise, SW1 Mode Switch SP3T, SW2 Roller Switch for Rotary Dial, SW3 Tactile Switch, SW4 Tactile Switch, SW5 Tactile Switch, SW6 Tactile Switch, SW7 Tactile Switch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

Commit message: made changes
Parts:
- removed T6, T7: ~, MyFootprints:CableClip_Harwin-S8101-46R, symbol MyLibrary:CableClip
Other:
- moved on the sheet: NT2, T4, T5
Changed lines of the file:
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@@
 	(symbol
 		(lib_id "Device:Net-Tie_2")
-		(at 551.815 334.645 0)
+		(at 549.91 344.17 0)
 		(unit 1)
 		(exclude_from_sim no)
@@
 		(dnp no)
 		(property "Reference" "NT2"
-			(at 551.815 330.0476 0)
+			(at 549.91 339.5726 0)
 			(effects
 				(font
@@
 		)
 		(property "Value" "Net-Tie_2"
-			(at 551.815 332.359 0)
+			(at 549.91 341.884 0)
 			(effects
 				(font
@@
 		)
 		(property "Footprint" "NetTie:NetTie-2_SMD_Pad0.5mm"
-			(at 551.815 334.645 0)
+			(at 549.91 344.17 0)
 			(effects
 				(font
@@
 		)
 		(property "Datasheet" "~"
-			(at 551.815 334.645 0)
-			(effects
-				(font
-					(size 1.27 1.27)
-				)
-				(hide yes)
-			)
-		)
-		(property "Description" ""
-			(at 551.815 334.645 0)
+			(at 549.91 344.17 0)
+			(effects
+				(font
+					(size 1.27 1.27)
+				)
+				(hide yes)
+			)
+		)
+		(property "Description" ""
+			(at 549.91 344.17 0)
 			(effects
 				(font
@@
 	(symbol
 		(lib_id "power:GND")
-		(at 549.275 334.645 0)
+		(at 547.37 344.17 0)
 		(unit 1)
 		(exclude_from_sim no)
@@
 		(dnp no)
 		(property "Reference" "#PWR0160"
-			(at 549.275 340.995 0)
+			(at 547.37 350.52 0)
 			(effects
 				(font
@@
 		)
 		(property "Value" "GND"
-			(at 549.402 339.0392 0)
+			(at 547.497 348.5642 0)
 			(effects
 				(font
@@
 		)
 		(property "Footprint" ""
-			(at 549.275 334.645 0)
+			(at 547.37 344.17 0)
 			(effects
 				(font
@@
 		)
 		(property "Datasheet" ""
-			(at 549.275 334.645 0)
-			(effects
-				(font
-					(size 1.27 1.27)
-				)
-				(hide yes)
-			)
-		)
-		(property "Description" ""
-			(at 549.275 334.645 0)
+			(at 547.37 344.17 0)
+			(effects
+				(font
+					(size 1.27 1.27)
+				)
+				(hide yes)
+			)
+		)
+		(property "Description" ""
+			(at 547.37 344.17 0)
 			(effects
 				(font
@@
 	(symbol
 		(lib_id "power:GNDA")
-		(at 554.355 334.645 0)
+		(at 552.45 344.17 0)
 		(unit 1)
 		(exclude_from_sim no)
@@
 		(dnp no)
 		(property "Reference" "#PWR0161"
-			(at 554.355 340.995 0)
+			(at 552.45 350.52 0)
 			(effects
 				(font
@@
 		)
 		(property "Value" "GNDA"
-			(at 554.482 339.0392 0)
+			(at 552.577 348.5642 0)
 			(effects
 				(font
@@
 		)
 		(property "Footprint" ""
-			(at 554.355 334.645 0)
+			(at 552.45 344.17 0)
 			(effects
 				(font
@@
 		)
 		(property "Datasheet" ""
-			(at 554.355 334.645 0)
-			(effects
-				(font
-					(size 1.27 1.27)
-				)
-				(hide yes)
-			)
-		)
-		(property "Description" ""
-			(at 554.355 334.645 0)
+			(at 552.45 344.17 0)
+			(effects
+				(font
+					(size 1.27 1.27)
+				)
+				(hide yes)
+			)
+		)
+		(property "Description" ""
+			(at 552.45 344.17 0)
 			(effects
 				(font
@@
 	)
 	(symbol
-		(lib_id "MyLibrary:CableClip")
-		(at 551.18 353.695 0)
-		(unit 1)
-		(exclude_from_sim no)
-		(in_bom yes)
-		(on_board yes)
-		(dnp no)
-		(property "Reference" "T7"
-			(at 553.085 354.33 0)
-			(effects
-				(font
-					(size 1.27 1.27)
-				)
-				(justify left)
-			)
-		)
-		(property "Value" "~"
-			(at 551.18 353.695 0)
-			(effects
-				(font
-					(size 1.27 1.27)
-				)
-			)
-		)
-		(property "Footprint" "MyFootprints:CableClip_Harwin-S8101-46R"
-			(at 551.18 353.695 0)
-			(effects
-				(font
-					(size 1.27 1.27)
-				)
-				(hide yes)
-			)
-		)
-		(property "Datasheet" ""
-			(at 551.18 353.695 0)
-			(effects
-				(font
-					(size 1.27 1.27)
-				)
-				(hide yes)
-			)
-		)
-		(property "Description" ""
-			(at 551.18 353.695 0)
-			(effects
-				(font
-					(size 1.27 1.27)
-				)
-				(hide yes)
-			)
-		)
-		(property "Mfg. Name" "Harwin"
-			(at 551.18 353.695 0)
-			(effects
-				(font
-					(size 1.27 1.27)
-				)
-				(hide yes)
-			)
-		)
-		(property "Mfg. Part No." "S8101-46R"
-			(at 551.18 356.235 0)
-			(effects
-				(font
-					(size 1.27 1.27)
-				)
-				(hide yes)
-			)
-		)
-		(instances
-			(project "RUSP_Mainboard"
-				(path "/f8b47531-6c06-4e54-9fc9-cd9d0f3dd69f"
-					(reference "T7")
-					(unit 1)
-				)
-			)
-		)
-	)
-	(symbol
 		(lib_id "power:GND")
 		(at 316.23 256.54 0)
@@
 	(symbol
 		(lib_id "MyLibrary:CableClip")
-		(at 551.18 346.71 0)
+		(at 549.275 356.235 0)
 		(unit 1)
 		(exclude_from_sim no)
@@
 		(dnp no)
 		(property "Reference" "T5"
-			(at 553.085 347.345 0)
+			(at 551.18 356.87 0)
 			(effects
 				(font
@@
 		)
 		(property "Value" "~"
-			(at 551.18 346.71 0)
+			(at 549.275 356.235 0)
 			(effects
 				(font
@@
 		)
 		(property "Footprint" "MyFootprints:CableClip_Harwin-S8101-46R"
-			(at 551.18 346.71 0)
+			(at 549.275 356.235 0)
 			(effects
 				(font
@@
 		)
 		(property "Datasheet" ""
-			(at 551.18 346.71 0)
-			(effects
-				(font
-					(size 1.27 1.27)
-				)
-				(hide yes)
-			)
-		)
-		(property "Description" ""
-			(at 551.18 346.71 0)
+			(at 549.275 356.235 0)
+			(effects
+				(font
+					(size 1.27 1.27)
+				)
+				(hide yes)
+			)
+		)
+		(property "Description" ""
+			(at 549.275 356.235 0)
 			(effects
 				(font
@@
 		)
 		(property "Mfg. Name" "Harwin"
-			(at 551.18 346.71 0)
+			(at 549.275 356.235 0)
 			(effects
 				(font
@@
 		)
 		(property "Mfg. Part No." "S8101-46R"
-			(at 551.18 349.25 0)
+			(at 549.275 358.775 0)
 			(effects
 				(font
@@
 	(symbol
 		(lib_id "MyLibrary:CableClip")
-		(at 551.18 342.9 0)
+		(at 549.275 352.425 0)
 		(unit 1)
 		(exclude_from_sim no)
@@
 		(dnp no)
 		(property "Reference" "T4"
-			(at 553.085 343.535 0)
+			(at 551.18 353.06 0)
 			(effects
 				(font
@@
 		)
 		(property "Value" "~"
-			(at 551.18 342.9 0)
+			(at 549.275 352.425 0)
 			(effects
 				(font
@@
 		)
 		(property "Footprint" "MyFootprints:CableClip_Harwin-S8101-46R"
-			(at 551.18 342.9 0)
+			(at 549.275 352.425 0)
 			(effects
 				(font
@@
 		)
 		(property "Datasheet" ""
-			(at 551.18 342.9 0)
-			(effects
-				(font
-					(size 1.27 1.27)
-				)
-				(hide yes)
-			)
-		)
-		(property "Description" ""
-			(at 551.18 342.9 0)
+			(at 549.275 352.425 0)
+			(effects
+				(font
+					(size 1.27 1.27)
+				)
+				(hide yes)
+			)
+		)
+		(property "Description" ""
+			(at 549.275 352.425 0)
 			(effects
 				(font
@@
 		)
 		(property "Mfg. Name" "Harwin"
-			(at 551.18 342.9 0)
+			(at 549.275 352.425 0)
 			(effects
 				(font
@@
 		)
 		(property "Mfg. Part No." "S8101-46R"
-			(at 551.18 345.44 0)
+			(at 549.275 354.965 0)
 			(effects
 				(font
@@
 					(unit 1)
 				)
-			)
-		)
-	)
-	(symbol
-		(lib_id "MyLibrary:CableClip")
-		(at 551.18 349.885 0)
-		(unit 1)
-		(exclude_from_sim no)
-		(in_bom yes)
-		(on_board yes)
-		(dnp no)
-		(property "Reference" "T6"
-			(at 553.085 350.52 0)
-			(effects
-				(font
-					(size 1.27 1.27)
-				)
-				(justify left)
-			)
-		)
-		(property "Value" "~"
-			(at 551.18 349.885 0)
-			(effects
-				(font
-					(size 1.27 1.27)
-				)
-			)
-		)
-		(property "Footprint" "MyFootprints:CableClip_Harwin-S8101-46R"
-			(at 551.18 349.885 0)
-			(effects
-				(font
-					(size 1.27 1.27)
-				)
-				(hide yes)
-			)
-		)
-		(property "Datasheet" ""
-			(at 551.18 349.885 0)
-			(effects
-				(font
-					(size 1.27 1.27)
-				)
-				(hide yes)
-			)
-		)
-		(property "Description" ""
-			(at 551.18 349.885 0)
-			(effects
-				(font
-					(size 1.27 1.27)
-				)
-				(hide yes)
-			)
-		)
-		(property "Mfg. Name" "Harwin"
-			(at 551.18 349.885 0)
-			(effects
-				(font
-					(size 1.27 1.27)
-				)
-				(hide yes)
-			)
-		)
-		(property "Mfg. Part No." "S8101-46R"
-			(at 551.18 352.425 0)
-			(effects
-				(font
-					(size 1.27 1.27)
-				)
-				(hide yes)
-			)
-		)
-		(instances
-			(project "RUSP_Mainboard"
-				(path "/f8b47531-6c06-4e54-9fc9-cd9d0f3dd69f"
-					(reference "T6")
-					(unit 1)
-				)

Commit message: for phase 1 prod
Parts:
- removed T4, T5: ~, MyFootprints:CableClip_Harwin-S8101-46R, symbol MyLibrary:CableClip
Changed lines of the file:
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@@
-	)
-	(symbol
-		(lib_id "MyLibrary:CableClip")
-		(at 549.275 356.235 0)
-		(unit 1)
-		(exclude_from_sim no)
-		(in_bom yes)
-		(on_board yes)
-		(dnp no)
-		(property "Reference" "T5"
-			(at 551.18 356.87 0)
-			(effects
-				(font
-					(size 1.27 1.27)
-				)
-				(justify left)
-			)
-		)
-		(property "Value" "~"
-			(at 549.275 356.235 0)
-			(effects
-				(font
-					(size 1.27 1.27)
-				)
-			)
-		)
-		(property "Footprint" "MyFootprints:CableClip_Harwin-S8101-46R"
-			(at 549.275 356.235 0)
-			(effects
-				(font
-					(size 1.27 1.27)
-				)
-				(hide yes)
-			)
-		)
-		(property "Datasheet" ""
-			(at 549.275 356.235 0)
-			(effects
-				(font
-					(size 1.27 1.27)
-				)
-				(hide yes)
-			)
-		)
-		(property "Description" ""
-			(at 549.275 356.235 0)
-			(effects
-				(font
-					(size 1.27 1.27)
-				)
-				(hide yes)
-			)
-		)
-		(property "Mfg. Name" "Harwin"
-			(at 549.275 356.235 0)
-			(effects
-				(font
-					(size 1.27 1.27)
-				)
-				(hide yes)
-			)
-		)
-		(property "Mfg. Part No." "S8101-46R"
-			(at 549.275 358.775 0)
-			(effects
-				(font
-					(size 1.27 1.27)
-				)
-				(hide yes)
-			)
-		)
-		(instances
-			(project "RUSP_Mainboard"
-				(path "/f8b47531-6c06-4e54-9fc9-cd9d0f3dd69f"
-					(reference "T5")
-					(unit 1)
-				)
-			)
-		)
-	)
-	(symbol
-		(lib_id "MyLibrary:CableClip")
-		(at 549.275 352.425 0)
-		(unit 1)
-		(exclude_from_sim no)
-		(in_bom yes)
-		(on_board yes)
-		(dnp no)
-		(property "Reference" "T4"
-			(at 551.18 353.06 0)
-			(effects
-				(font
-					(size 1.27 1.27)
-				)
-				(justify left)
-			)
-		)
-		(property "Value" "~"
-			(at 549.275 352.425 0)
-			(effects
-				(font
-					(size 1.27 1.27)
-				)
-			)
-		)
-		(property "Footprint" "MyFootprints:CableClip_Harwin-S8101-46R"
-			(at 549.275 352.425 0)
-			(effects
-				(font
-					(size 1.27 1.27)
-				)
-				(hide yes)
-			)
-		)
-		(property "Datasheet" ""
-			(at 549.275 352.425 0)
-			(effects
-				(font
-					(size 1.27 1.27)
-				)
-				(hide yes)
-			)
-		)
-		(property "Description" ""
-			(at 549.275 352.425 0)
-			(effects
-				(font
-					(size 1.27 1.27)
-				)
-				(hide yes)
-			)
-		)
-		(property "Mfg. Name" "Harwin"
-			(at 549.275 352.425 0)
-			(effects
-				(font
-					(size 1.27 1.27)
-				)
-				(hide yes)
-			)
-		)
-		(property "Mfg. Part No." "S8101-46R"
-			(at 549.275 354.965 0)
-			(effects
-				(font
-					(size 1.27 1.27)
-				)
-				(hide yes)
-			)
-		)
-		(instances
-			(project "RUSP_Mainboard"
-				(path "/f8b47531-6c06-4e54-9fc9-cd9d0f3dd69f"
-					(reference "T4")
-					(unit 1)
-				)
-			)
-		)
 	)
 	(symbol
